Commit message: Robot can be control by TeleopKey method and gripper handling also config to the keyboard.

File: urdf/myrobotOLD.urdf (robot description, URDF)
Before this commit: robot pde4430_cw2_robot_new, 5 links, 4 joints
Links:
- link left_gripper: mass 0.5 -> 1.86518207129963
- link right_gripper: mass 0.15 -> 1.61587084761863

File: urdf/myrobot_test.urdf (robot description, URDF)
Before this commit: robot pde4430_cw2_robot_new, 5 links, 4 joints
Links:
- link left_gripper: mass 0.5 -> 1.86518207129963
- link right_gripper: mass 0.15 -> 1.61587084761863
