Commit message: Added trasmission and hardware_interface for each joint

File: urdf/myrobot.urdf (robot description, URDF)
Before this commit: robot pde4430_cw2_robot_new, 6 links, 5 joints
Links:
- removed link map
- link chassy: geometry collision mesh filename=package://pde4430_cw2_robot_description/meshes/chassy.STL; visual mesh filename=package://pde4430_cw2_robot_description/meshes/chassy.STL
- link left_gripper: geometry collision mesh filename=package://pde4430_cw2_robot_description/meshes/left_gripper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; visual mesh filename=package://pde4430_cw2_robot_description/meshes/left_gripper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
- link left_wheel: geometry collision mesh filename=package://pde4430_cw2_robot_description/meshes/left_wheel.S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; visual mesh filename=package://pde4430_cw2_robot_description/meshes/left_wheel.S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
- link right_gripper: geometry collision mesh filename=package://pde4430_cw2_robot_description/meshes/right_grippe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; visual mesh filename=package://pde4430_cw2_robot_description/meshes/right_grippe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
- link right_wheel: geometry collision mesh filename=package://pde4430_cw2_robot_description/meshes/right_wheel.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; visual mesh filename=package://pde4430_cw2_robot_description/meshes/right_wheel.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
Joints:
- removed joint map_to_chassy
- joint left_gripper_joint: limit lower=0.61 upper=-0.78 effort=10 velocity=5 -> lower=-0.78 upper=0.61 effort=10 velocity=5

Commit message: Using cmd_vel robot can move. For now only wheels can operate. Using teleop and normal myrobot.py file can operate the robot

File: urdf/myrobot.urdf (robot description, URDF)
Before this commit: robot pde4430_cw2_robot_new, 5 links, 4 joints
Joints:
- joint right_wheel_joint: axis 0 1 0 -> 0 -1 0

Commit message: updated README file and URDF file

File: urdf/myrobot.urdf (robot description, URDF)
Before this commit: robot pde4430_cw2_robot_new, 5 links, 4 joints
Links:
- link left_gripper: mass 0.5 -> 0.65
- link left_wheel: mass 1.16602182282338 -> 2.16602182282338
- link right_gripper: mass 0.15 -> 0.65
- link right_wheel: mass 1.16602182282338 -> 2.16602182282338
Joints:
- joint left_gripper_joint: limit lower=-0.78 upper=0.61 effort=10 velocity=5 -> lower=-0.78 upper=0.61 effort=20 velocity=1
- joint right_gripper_joint: limit lower=-0.78 upper=0.61 effort=10 velocity=5 -> lower=-0.78 upper=0.61 effort=20 velocity=1

Commit message: Lidar fixed and working.

File: urdf/myrobot.urdf (robot description, URDF)
Before this commit: robot pde4430_cw2_robot_new, 5 links, 4 joints
Links:
- added link lidar_link, mass 1.0; collision mesh filename=package://pde4430_cw2_robot_description/meshes/lidar.STL; visual mesh filename=package://pde4430_cw2_robot_description/meshes/lidar.STL
- link left_gripper: mass 0.65 -> 0.15
- link right_gripper: mass 0.65 -> 0.15
Joints:
- added joint lidar_joint: type fixed, parent chassy, child lidar_link, origin xyz=0.19007 -0.35181 0.16761 rpy=1.5708 0 0, axis 0 0 0

Commit message: README file updated. Commit and push the developed status for CW2 submission.

File: urdf/myrobot.urdf (robot description, URDF)
Before this commit: robot pde4430_cw2_robot_new, 6 links, 5 joints
Joints:
- joint lidar_joint: origin xyz=0.19007 -0.35181 0.16761 rpy=1.5708 0 0 -> xyz=0.19007 -0.35181 0.16761 rpy=0 0 0
